File: eagle/FedorBall/FedorBall.brd (EAGLE design)
At the start: 100 x 80 mm, 18 parts, among them IC1 MEGA16-P, IC2 7805T, X1 22-23-2041, X2 22-23-2041

Commit message: update schematic and board according to last hardware experiments
Parts:
- removed R3, R4: 10k, rcl:0207/10
- added CRYSTAL_16MHZ: (no value), crystal:DIL08S
- moved R2 117.8 mm to (6.35, -3.81), flipped to the top
Connections:
- removed net GSCLK: IC1.21, LED_DRIVER.7
- removed net MISO_10K: LED_DRIVER.8, R3.1
- removed net MOSI_10K: LED_DRIVER.9, R4.1
- removed net N$5: IC1.6, ISP.1, R4.2
- removed net N$7: IC1.8, ISP.7, R2.2
- removed net N$8: IC1.7, ISP.9, R3.2
- removed net SCK_10K: LED_DRIVER.10, R2.1
- new net 16MHZ_CLK: CRYSTAL_16MHZ.5, IC1.13, LED_DRIVER.7
- new net MISO: IC1.7, ISP.9, LED_DRIVER.8
- new net MOSI: IC1.6, ISP.1, LED_DRIVER.9
- new net SCK: IC1.8, ISP.7, LED_DRIVER.10
- net +5V: now also CRYSTAL_16MHZ.8, R2.1
- net BLANK: now also R2.2
- net GND: now also CRYSTAL_16MHZ.4, S1.P$2
- net N$6: now also S1.P$4
Changed lines of the file:
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@@
 <element name="C7" library="rcl" package="C050-024X044" value="0.1u" x="86.36" y="30.48" rot="MR180"/>
 <element name="C8" library="rcl" package="C050-024X044" value="47u" x="86.36" y="22.86" rot="MR180"/>
-<element name="R2" library="rcl" package="0207/10" value="10k" x="93.98" y="74.93" rot="MR0"/>
-<element name="R3" library="rcl" package="0207/10" value="10k" x="92.71" y="68.58" rot="MR0"/>
-<element name="R4" library="rcl" package="0207/10" value="10k" x="87.63" y="7.62" rot="MR0"/>
 <element name="ISP" library="SparkFun" package="2X5-SHROUDED" value="M05X2SHD" x="62.23" y="66.04" rot="MR180"/>
 <element name="LED_DRIVER" library="SparkFun" package="2X5-SHROUDED" value="M05X2SHD" x="93.98" y="54.61" rot="MR180"/>
 <element name="R5" library="rcl" package="0207/10" value="10k" x="8.89" y="10.16" rot="MR180"/>
 <element name="R6" library="rcl" package="0207/10" value="10k" x="8.89" y="3.81" rot="MR180"/>
+<element name="R2" library="rcl" package="0207/10" value="10k" x="6.35" y="-3.81"/>
+<element name="CRYSTAL_16MHZ" library="crystal" package="DIL08S" value="" x="-7.62" y="2.54">
+<attribute name="OC_NEWARK" value="unknown" x="-7.62" y="2.54" size="1.778" layer="27" display="off"/>
+<attribute name="MPN" value="" x="-7.62" y="2.54" size="1.778" layer="27" display="off"/>
+<attribute name="MF" value="" x="-7.62" y="2.54" size="1.778" layer="27" display="off"/>
+<attribute name="OC_FARNELL" value="unknown" x="-7.62" y="2.54" size="1.778" layer="27" display="off"/>
+</element>
 </elements>
 <signals>
@@
 <contactref element="LED_DRIVER" pad="2"/>
 <contactref element="LED_DRIVER" pad="4"/>
+<contactref element="R2" pad="1"/>
+<contactref element="CRYSTAL_16MHZ" pad="8"/>
 <wire x1="95.25" y1="49.53" x2="95.25" y2="52.07" width="0" layer="19" extent="1-1"/>
 <wire x1="83.82" y1="30.48" x2="95.25" y2="49.53" width="0" layer="19" extent="1-1"/>
@@
 <wire x1="3.81" y1="10.16" x2="8.89" y2="15.24" width="0" layer="19" extent="1-1"/>
 <wire x1="3.81" y1="3.81" x2="3.81" y2="10.16" width="0" layer="19" extent="1-1"/>
+<wire x1="1.27" y1="-3.81" x2="3.81" y2="3.81" width="0" layer="19" extent="1-1"/>
+<wire x1="-11.43" y1="6.35" x2="3.81" y2="3.81" width="0" layer="19" extent="1-1"/>
 <wire x1="7.62" y1="33.02" x2="8.89" y2="15.24" width="0" layer="19" extent="1-1"/>
 </signal>
@@
 <contactref element="LED_DRIVER" pad="1"/>
 <contactref element="ISP" pad="6"/>
+<contactref element="CRYSTAL_16MHZ" pad="4"/>
+<contactref element="CRYSTAL_16MHZ" pad="4"/>
+<contactref element="S1" pad="P$2"/>
 <wire x1="87.63" y1="38.1" x2="92.71" y2="49.53" width="0" layer="19" extent="1-1"/>
 <wire x1="88.9" y1="30.48" x2="87.63" y2="38.1" width="0" layer="19" extent="1-1"/>
@@
 <wire x1="10.16" y1="33.02" x2="30.48" y2="46.99" width="0" layer="19" extent="1-1"/>
 <wire x1="8.89" y1="17.78" x2="10.16" y2="33.02" width="0" layer="19" extent="1-1"/>
-<wire x1="30.48" y1="11.43" x2="8.89" y2="17.78" width="0" layer="19" extent="1-1"/>
+<wire x1="22.86" y1="11.43" x2="8.89" y2="17.78" width="0" layer="19" extent="1-1"/>
+<wire x1="30.48" y1="11.43" x2="22.86" y2="11.43" width="0" layer="19" extent="1-1"/>
+<wire x1="-3.81" y1="-1.27" x2="8.89" y2="17.78" width="0" layer="19" extent="1-1"/>
 <wire x1="63.5" y1="66.04" x2="50.8" y2="44.45" width="0" layer="19" extent="1-1"/>
 <wire x1="63.5" y1="68.58" x2="63.5" y2="66.04" width="0" layer="19" extent="1-1"/>
@@
 <wire x1="30.48" y1="52.07" x2="35.56" y2="49.53" width="0" layer="19" extent="1-16"/>
 </signal>
-<signal name="N$5">
+<signal name="MOSI">
 <contactref element="IC1" pad="6"/>
-<contactref element="R4" pad="2"/>
 <contactref element="ISP" pad="1"/>
-<wire x1="82.55" y1="7.62" x2="60.96" y2="60.96" width="0" layer="19" extent="1-1"/>
+<contactref element="LED_DRIVER" pad="9"/>
+<wire x1="60.96" y1="60.96" x2="92.71" y2="59.69" width="0" layer="19" extent="1-1"/>
 <wire x1="50.8" y1="57.15" x2="60.96" y2="60.96" width="0" layer="19" extent="1-1"/>
 </signal>
-<signal name="N$7">
+<signal name="SCK">
 <contactref element="IC1" pad="8"/>
-<contactref element="R2" pad="2"/>
 <contactref element="ISP" pad="7"/>
-<wire x1="88.9" y1="74.93" x2="60.96" y2="68.58" width="0" layer="19" extent="1-1"/>
-<wire x1="50.8" y1="52.07" x2="88.9" y2="74.93" width="0" layer="19" extent="1-1"/>
-</signal>
-<signal name="N$8">
+<contactref element="LED_DRIVER" pad="10"/>
+<wire x1="60.96" y1="68.58" x2="95.25" y2="59.69" width="0" layer="19" extent="1-1"/>
+<wire x1="50.8" y1="52.07" x2="60.96" y2="68.58" width="0" layer="19" extent="1-1"/>
+</signal>
+<signal name="MISO">
 <contactref element="IC1" pad="7"/>
-<contactref element="R3" pad="2"/>
 <contactref element="ISP" pad="9"/>
-<wire x1="87.63" y1="68.58" x2="60.96" y2="71.12" width="0" layer="19" extent="1-1"/>
-<wire x1="50.8" y1="54.61" x2="87.63" y2="68.58" width="0" layer="19" extent="1-1"/>
+<contactref element="LED_DRIVER" pad="8"/>
+<wire x1="60.96" y1="71.12" x2="95.25" y2="57.15" width="0" layer="19" extent="1-1"/>
+<wire x1="50.8" y1="54.61" x2="60.96" y2="71.12" width="0" layer="19" extent="1-1"/>
 </signal>
 <signal name="N$6">
@@
 <contactref element="S1" pad="P$3"/>
 <contactref element="ISP" pad="5"/>
+<contactref element="S1" pad="P$4"/>
+<wire x1="50.8" y1="49.53" x2="60.96" y2="66.04" width="0" layer="19" extent="1-1"/>
+<wire x1="57.15" y1="45.72" x2="50.8" y2="49.53" width="0" layer="19" extent="1-1"/>
 <wire x1="60.96" y1="44.45" x2="57.15" y2="45.72" width="0" layer="19" extent="1-1"/>
-<wire x1="50.8" y1="49.53" x2="57.15" y2="45.72" width="0" layer="19" extent="1-1"/>
-<wire x1="30.48" y1="6.35" x2="50.8" y2="49.53" width="0" layer="19" extent="1-1"/>
-<wire x1="60.96" y1="66.04" x2="30.48" y2="6.35" width="0" layer="19" extent="1-1"/>
+<wire x1="30.48" y1="6.35" x2="57.15" y2="45.72" width="0" layer="19" extent="1-1"/>
+<wire x1="22.86" y1="6.35" x2="30.48" y2="6.35" width="0" layer="19" extent="1-1"/>
 </signal>
 <signal name="N$9">
@@
 <contactref element="LED_DRIVER" pad="6"/>
 <contactref element="IC1" pad="18"/>
+<contactref element="R2" pad="2"/>
 <wire x1="50.8" y1="26.67" x2="95.25" y2="54.61" width="0" layer="19" extent="1-1"/>
-</signal>
-<signal name="GSCLK">
-<contactref element="LED_DRIVER" pad="7"/>
-<contactref element="IC1" pad="21"/>
-<wire x1="35.56" y1="21.59" x2="92.71" y2="57.15" width="0" layer="19" extent="1-1"/>
+<wire x1="11.43" y1="-3.81" x2="50.8" y2="26.67" width="0" layer="19" extent="1-1"/>
 </signal>
 <signal name="VPRG">
@@
 <wire x1="50.8" y1="24.13" x2="92.71" y2="52.07" width="0" layer="19" extent="1-1"/>
 </signal>
-<signal name="SCK_10K">
-<contactref element="R2" pad="1"/>
-<contactref element="LED_DRIVER" pad="10"/>
-<wire x1="95.25" y1="59.69" x2="99.06" y2="74.93" width="0" layer="19" extent="1-1"/>
-</signal>
-<signal name="MISO_10K">
-<contactref element="R3" pad="1"/>
-<contactref element="LED_DRIVER" pad="8"/>
-<wire x1="95.25" y1="57.15" x2="97.79" y2="68.58" width="0" layer="19" extent="1-1"/>
-</signal>
-<signal name="MOSI_10K">
-<contactref element="R4" pad="1"/>
-<contactref element="LED_DRIVER" pad="9"/>
-<wire x1="92.71" y1="7.62" x2="92.71" y2="59.69" width="0" layer="19" extent="1-1"/>
+<signal name="16MHZ_CLK">
+<contactref element="CRYSTAL_16MHZ" pad="5"/>
+<contactref element="IC1" pad="13"/>
+<contactref element="LED_DRIVER" pad="7"/>
+<wire x1="50.8" y1="39.37" x2="92.71" y2="57.15" width="0" layer="19" extent="1-1"/>
+<wire x1="-3.81" y1="6.35" x2="50.8" y2="39.37" width="0" layer="19" extent="1-1"/>
 </signal>
 </signals>

Commit message: minor scheme changes
Connections:
- net INT0: now also IC1.16; no longer IC1.17
- net INT1: now also IC1.17; no longer IC1.16
Changed lines of the file:
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@@
 </signal>
 <signal name="INT1">
-<contactref element="IC1" pad="16"/>
 <contactref element="X1" pad="3"/>
-<wire x1="8.89" y1="20.32" x2="50.8" y2="31.75" width="0" layer="19" extent="1-1"/>
+<contactref element="IC1" pad="17"/>
+<wire x1="8.89" y1="20.32" x2="50.8" y2="29.21" width="0" layer="19" extent="1-1"/>
 </signal>
 <signal name="INT0">
-<contactref element="IC1" pad="17"/>
 <contactref element="X1" pad="4"/>
-<wire x1="8.89" y1="22.86" x2="50.8" y2="29.21" width="0" layer="19" extent="1-1"/>
+<contactref element="IC1" pad="16"/>
+<wire x1="8.89" y1="22.86" x2="50.8" y2="31.75" width="0" layer="19" extent="1-1"/>
 </signal>
 <signal name="XLAT">
